File: SD_Card_Adapter-VCU128.kicad_pcb (KiCad board)
At the start: 2 copper layers, 61 x 70.1 mm, 45 parts, among them J1 ASP-184330-01, J2 87834-1011, J3 GSD090012SEU, Q1 SI1012R-T1-GE3, U1 TXB0108DQSR, U2 TXB0108DQSR

Commit message: Revision B.
All signals have been moved to row H of FMC+ connector J1
because the ones in row M are connected to FPGA pins that
are dedicated to high speed transceivers.
Parts:
- moved R2 1.14 mm to (106.0, 83.2)
- moved R3 0.51 mm to (101.6, 83.2)
Connections:
- J1 pad H04: unconnected-(J1-PadH04) -> TCK_LS
- J1 pad H07: unconnected-(J1-PadH07) -> TMS_LS
- J1 pad H10: unconnected-(J1-PadH10) -> TDO_LS
- J1 pad H11: unconnected-(J1-PadH11) -> TDI_LS
- J1 pad H13: unconnected-(J1-PadH13) -> RST_LS
- J1 pad H16: unconnected-(J1-PadH16) -> PROTECT
- J1 pad H17: unconnected-(J1-PadH17) -> DETECT
- J1 pad H19: unconnected-(J1-PadH19) -> SDIO_DAT1_LS
- J1 pad H22: unconnected-(J1-PadH22) -> SDIO_DAT0_LS
- J1 pad H25: unconnected-(J1-PadH25) -> SDIO_CLK_LS
- J1 pad H31: unconnected-(J1-PadH31) -> SDIO_CMD_LS
- J1 pad H34: unconnected-(J1-PadH34) -> SDIO_CD_DAT3_LS
- J1 pad H37: unconnected-(J1-PadH37) -> SDIO_DAT2_LS
- J1 pad M02: TMS_LS -> unconnected-(J1-PadM02)
- J1 pad M03: TCK_LS -> unconnected-(J1-PadM03)
- J1 pad M06: TDO_LS -> unconnected-(J1-PadM06)
- J1 pad M07: TDI_LS -> unconnected-(J1-PadM07)
- J1 pad M10: RST_LS -> unconnected-(J1-PadM10)
- J1 pad M14: PROTECT -> unconnected-(J1-PadM14)
- J1 pad M15: DETECT -> unconnected-(J1-PadM15)
- J1 pad M18: SDIO_DAT1_LS -> unconnected-(J1-PadM18)
- J1 pad M22: SDIO_DAT0_LS -> unconnected-(J1-PadM22)
- J1 pad M26: SDIO_CLK_LS -> unconnected-(J1-PadM26)
- J1 pad M30: SDIO_CMD_LS -> unconnected-(J1-PadM30)
- J1 pad M34: SDIO_CD_DAT3_LS -> unconnected-(J1-PadM34)
- J1 pad M38: SDIO_DAT2_LS -> unconnected-(J1-PadM38)
Routing:
- net TMS_LS: track 19.3 -> 31.4 mm
- net +1V8: track 86.8 -> 96.8 mm, vias 3 -> 9
- net TDO_LS: track 15.6 -> 22.8 mm
- net SDIO_CD_DAT3_LS: track 7.05 -> 13.4 mm, vias 1 -> 2
- net SDIO_CLK_LS: track 9.87 -> 15.5 mm, vias 1 -> 2
- net PROTECT: track 29.0 -> 34.6 mm, vias 2 -> 3
- net SDIO_DAT2_LS: track 10.2 -> 15.7 mm, vias 1 -> 2
- net TCK_LS: track 16.2 -> 21.5 mm
- net SDIO_CMD_LS: track 8.44 -> 13.5 mm, vias 1 -> 2
- net SDIO_DAT0_LS: track 13.7 -> 18.5 mm, vias 1 -> 2
- net SDIO_DAT1_LS: track 19.4 -> 23.9 mm, vias 1 -> 2
- net RST_LS: track 19.6 -> 24.0 mm
- net TDI_LS: track 17.4 -> 21.8 mm
- net DETECT: track 28.9 -> 32.9 mm, vias 2 -> 3
- net GND: vias 77 -> 76
Other:
- board text added: "FMC+ Daughterboard: SD Card Reader + JTAG Header -- Rev. B"
- board text removed: "FMC+ Daughterboard: SD Card Reader + JTAG Header"
