File: SD_Card_Adapter-VCU128.kicad_sch (KiCad schematic)
At the start: 45 parts, among them J1 ASP-184330-01, J2 87834-1011, J3 GSD090012SEU, Q1 SI1012R-T1-GE3, U1 TXB0108DQSR, U2 TXB0108DQSR

Commit message: Revision B.
All signals have been moved to row H of FMC+ connector J1
because the ones in row M are connected to FPGA pins that
are dedicated to high speed transceivers.
Connections:
- net DETECT: now also J1.H17; no longer J1.M15
- net PROTECT: now also J1.H16; no longer J1.M14
- net RST_LS: now also J1.H13; no longer J1.M10
- net SDIO_CD_DAT3_LS: now also J1.H34; no longer J1.M34
- net SDIO_CLK_LS: now also J1.H25; no longer J1.M26
- net SDIO_CMD_LS: now also J1.H31; no longer J1.M30
- net SDIO_DAT0_LS: now also J1.H22; no longer J1.M22
- net SDIO_DAT1_LS: now also J1.H19; no longer J1.M18
- net SDIO_DAT2_LS: now also J1.H37; no longer J1.M38
- net TCK_LS: now also J1.H04; no longer J1.M03
- net TDI_LS: now also J1.H11; no longer J1.M07
- net TDO_LS: now also J1.H10; no longer J1.M06
- net TMS_LS: now also J1.H07; no longer J1.M02
Other:
- moved on the sheet: J1F
